File: kicad_project/CP70_preamp/CP70_preamp.kicad_pcb (KiCad board)
At the start: 0 parts

Commit message: design of 16 channel pre amp, including circuit board, ordered. Gerbers in repository.
Parts:
- added C201: 220 nF / 50 V, Capacitor_THT:C_Disc_D6.0mm_W2.5mm_P5.00mm, F.Cu at (158.3, 144.0)
- added C202: 220 nF / 50 V, Capacitor_THT:C_Disc_D6.0mm_W2.5mm_P5.00mm, F.Cu at (197.0, 143.3)
- added C203: 220 nF / 50 V, Capacitor_THT:C_Disc_D6.0mm_W2.5mm_P5.00mm, F.Cu at (197.0, 84.3)
- added C204: 220 nF / 50 V, Capacitor_THT:C_Disc_D6.0mm_W2.5mm_P5.00mm, F.Cu at (158.2, 83.7)
- added C205: 100uF / 35V, Capacitor_THT:CP_Radial_D10.0mm_P5.00mm, F.Cu at (140.9, 68.4)
- added C207: 100uF / 35V, Capacitor_THT:CP_Radial_D10.0mm_P5.00mm, F.Cu at (180.2, 68.4)
- added D201: LED green 5 mm, LED_THT:LED_D5.0mm, F.Cu at (166.3, 64.8)
- added D202: LED green 5 mm, LED_THT:LED_D5.0mm, F.Cu at (152.9, 64.8)
- added H201: MountingHole_Pad, MountingHole:MountingHole_3.2mm_M3_Pad_Via, F.Cu at (129.0, 60.0)
- added H202: MountingHole_Pad, MountingHole:MountingHole_3.2mm_M3_Pad_Via, F.Cu at (129.0, 148.0)
- added H203: MountingHole_Pad, MountingHole:MountingHole_3.2mm_M3_Pad_Via, F.Cu at (235.0, 60.0)
- added H204: MountingHole_Pad, MountingHole:MountingHole_3.2mm_M3_Pad_Via, F.Cu at (235.0, 148.0)
- added J201: Conn_01x03_Socket, Connector_Phoenix_MSTB:PhoenixContact_MSTBVA_2,5_3-G-5,08_1x03_P5.08mm_Vertical, F.Cu at (203.1, 68.3)
- added J202: Conn_02x20_Odd_Even, Connector_IDC:IDC-Header_2x20_P2.54mm_Latch_Horizontal, F.Cu at (219.6, 81.1)
- added J203: Conn_01x08, Connector_PinHeader_2.54mm:PinHeader_1x08_P2.54mm_Vertical, F.Cu at (110.0, 59.0)
- added J204: Conn_01x08, Connector_PinHeader_2.54mm:PinHeader_1x08_P2.54mm_Vertical, F.Cu at (115.1, 59.0)
- added J205: Conn_01x08, Connector_PinHeader_2.54mm:PinHeader_1x08_P2.54mm_Vertical, F.Cu at (110.0, 83.1)
- added J206: Conn_01x08, Connector_PinHeader_2.54mm:PinHeader_1x08_P2.54mm_Vertical, F.Cu at (115.1, 83.1)
- added J207: Conn_01x08, Connector_PinHeader_2.54mm:PinHeader_1x08_P2.54mm_Vertical, F.Cu at (110.0, 107.2)
- added J208: Conn_01x08, Connector_PinHeader_2.54mm:PinHeader_1x08_P2.54mm_Vertical, F.Cu at (115.1, 107.2)
- added J209: Conn_01x08, Connector_PinHeader_2.54mm:PinHeader_1x08_P2.54mm_Vertical, F.Cu at (110.0, 131.4)
- added J210: Conn_01x08, Connector_PinHeader_2.54mm:PinHeader_1x08_P2.54mm_Vertical, F.Cu at (115.1, 131.4)
- added R201: 2K7, Resistor_THT:R_Axial_DIN0207_L6.3mm_D2.5mm_P7.62mm_Horizontal, F.Cu at (162.5, 72.4)
- added R202: 2K7, Resistor_THT:R_Axial_DIN0207_L6.3mm_D2.5mm_P7.62mm_Horizontal, F.Cu at (149.1, 72.4)
- added R203: 470K, Resistor_THT:R_Axial_DIN0207_L6.3mm_D2.5mm_P7.62mm_Horizontal, F.Cu at (124.3, 68.1)
- added R204: 470K, Resistor_THT:R_Axial_DIN0207_L6.3mm_D2.5mm_P7.62mm_Horizontal, F.Cu at (124.3, 72.8)
- added R205: 470K, Resistor_THT:R_Axial_DIN0207_L6.3mm_D2.5mm_P7.62mm_Horizontal, F.Cu at (124.3, 77.5)
- added R206: 470K, Resistor_THT:R_Axial_DIN0207_L6.3mm_D2.5mm_P7.62mm_Horizontal, F.Cu at (124.3, 82.3)
- added R207: 470K, Resistor_THT:R_Axial_DIN0207_L6.3mm_D2.5mm_P7.62mm_Horizontal, F.Cu at (124.3, 87.0)
- added R208: 470K, Resistor_THT:R_Axial_DIN0207_L6.3mm_D2.5mm_P7.62mm_Horizontal, F.Cu at (124.3, 91.7)
- added R209: 470K, Resistor_THT:R_Axial_DIN0207_L6.3mm_D2.5mm_P7.62mm_Horizontal, F.Cu at (124.3, 96.5)
- added R210: 470K, Resistor_THT:R_Axial_DIN0207_L6.3mm_D2.5mm_P7.62mm_Horizontal, F.Cu at (124.3, 101.2)
- added R211: 100R, Resistor_THT:R_Axial_DIN0207_L6.3mm_D2.5mm_P7.62mm_Horizontal, F.Cu at (146.8, 95.1)
- added R212: 100R, Resistor_THT:R_Axial_DIN0207_L6.3mm_D2.5mm_P7.62mm_Horizontal, F.Cu at (146.8, 100.2)
- added R213: 100R, Resistor_THT:R_Axial_DIN0207_L6.3mm_D2.5mm_P7.62mm_Horizontal, F.Cu at (146.8, 109.1)
- added R214: 100R, Resistor_THT:R_Axial_DIN0207_L6.3mm_D2.5mm_P7.62mm_Horizontal, F.Cu at (146.8, 114.1)
- added R215: 100R, Resistor_THT:R_Axial_DIN0207_L6.3mm_D2.5mm_P7.62mm_Horizontal, F.Cu at (146.8, 122.4)
- added R216: 100R, Resistor_THT:R_Axial_DIN0207_L6.3mm_D2.5mm_P7.62mm_Horizontal, F.Cu at (146.8, 127.5)
- added R217: 100R, Resistor_THT:R_Axial_DIN0207_L6.3mm_D2.5mm_P7.62mm_Horizontal, F.Cu at (146.8, 135.7)
- added R218: 100R, Resistor_THT:R_Axial_DIN0207_L6.3mm_D2.5mm_P7.62mm_Horizontal, F.Cu at (146.8, 140.8)
- added R219: 100R, Resistor_THT:R_Axial_DIN0207_L6.3mm_D2.5mm_P7.62mm_Horizontal, F.Cu at (172.2, 90.0)
- added R220: 100R, Resistor_THT:R_Axial_DIN0207_L6.3mm_D2.5mm_P7.62mm_Horizontal, F.Cu at (172.2, 95.1)
- added R221: 100R, Resistor_THT:R_Axial_DIN0207_L6.3mm_D2.5mm_P7.62mm_Horizontal, F.Cu at (172.2, 104.0)
- added R222: 100R, Resistor_THT:R_Axial_DIN0207_L6.3mm_D2.5mm_P7.62mm_Horizontal, F.Cu at (172.2, 109.1)
- added R223: 100R, Resistor_THT:R_Axial_DIN0207_L6.3mm_D2.5mm_P7.62mm_Horizontal, F.Cu at (172.2, 117.3)
- added R224: 100R, Resistor_THT:R_Axial_DIN0207_L6.3mm_D2.5mm_P7.62mm_Horizontal, F.Cu at (172.2, 122.4)
- added R225: 100R, Resistor_THT:R_Axial_DIN0207_L6.3mm_D2.5mm_P7.62mm_Horizontal, F.Cu at (172.2, 130.7)
- added R226: 100R, Resistor_THT:R_Axial_DIN0207_L6.3mm_D2.5mm_P7.62mm_Horizontal, F.Cu at (172.2, 135.7)
- added R227: 470K, Resistor_THT:R_Axial_DIN0207_L6.3mm_D2.5mm_P7.62mm_Horizontal, F.Cu at (124.3, 105.9)
- added R228: 470K, Resistor_THT:R_Axial_DIN0207_L6.3mm_D2.5mm_P7.62mm_Horizontal, F.Cu at (124.3, 110.7)
- added R229: 470K, Resistor_THT:R_Axial_DIN0207_L6.3mm_D2.5mm_P7.62mm_Horizontal, F.Cu at (124.3, 115.4)
- added R230: 470K, Resistor_THT:R_Axial_DIN0207_L6.3mm_D2.5mm_P7.62mm_Horizontal, F.Cu at (124.3, 120.2)
- added R231: 470K, Resistor_THT:R_Axial_DIN0207_L6.3mm_D2.5mm_P7.62mm_Horizontal, F.Cu at (124.3, 124.9)
- added R232: 470K, Resistor_THT:R_Axial_DIN0207_L6.3mm_D2.5mm_P7.62mm_Horizontal, F.Cu at (124.3, 129.6)
- added R233: 470K, Resistor_THT:R_Axial_DIN0207_L6.3mm_D2.5mm_P7.62mm_Horizontal, F.Cu at (124.3, 134.4)
- added R234: 470K, Resistor_THT:R_Axial_DIN0207_L6.3mm_D2.5mm_P7.62mm_Horizontal, F.Cu at (124.3, 139.1)
- added R235: 100R, Resistor_THT:R_Axial_DIN0207_L6.3mm_D2.5mm_P7.62mm_Horizontal, F.Cu at (186.2, 95.7)
- added R236: 100R, Resistor_THT:R_Axial_DIN0207_L6.3mm_D2.5mm_P7.62mm_Horizontal, F.Cu at (186.2, 100.8)
- added R237: 100R, Resistor_THT:R_Axial_DIN0207_L6.3mm_D2.5mm_P7.62mm_Horizontal, F.Cu at (186.2, 109.1)
- added R238: 100R, Resistor_THT:R_Axial_DIN0207_L6.3mm_D2.5mm_P7.62mm_Horizontal, F.Cu at (186.2, 114.1)
- added R239: 100R, Resistor_THT:R_Axial_DIN0207_L6.3mm_D2.5mm_P7.62mm_Horizontal, F.Cu at (186.2, 122.4)
- added R240: 100R, Resistor_THT:R_Axial_DIN0207_L6.3mm_D2.5mm_P7.62mm_Horizontal, F.Cu at (186.2, 128.7)
- added R241: 100R, Resistor_THT:R_Axial_DIN0207_L6.3mm_D2.5mm_P7.62mm_Horizontal, F.Cu at (186.2, 135.7)
- added R242: 100R, Resistor_THT:R_Axial_DIN0207_L6.3mm_D2.5mm_P7.62mm_Horizontal, F.Cu at (186.2, 142.1)
- added R243: 100R, Resistor_THT:R_Axial_DIN0207_L6.3mm_D2.5mm_P7.62mm_Horizontal, F.Cu at (211.0, 90.6)
- added R244: 100R, Resistor_THT:R_Axial_DIN0207_L6.3mm_D2.5mm_P7.62mm_Horizontal, F.Cu at (211.0, 95.7)
- added R245: 100R, Resistor_THT:R_Axial_DIN0207_L6.3mm_D2.5mm_P7.62mm_Horizontal, F.Cu at (211.0, 104.0)
- added R246: 100R, Resistor_THT:R_Axial_DIN0207_L6.3mm_D2.5mm_P7.62mm_Horizontal, F.Cu at (211.0, 109.1)
- added R247: 100R, Resistor_THT:R_Axial_DIN0207_L6.3mm_D2.5mm_P7.62mm_Horizontal, F.Cu at (211.0, 117.3)
- added R248: 100R, Resistor_THT:R_Axial_DIN0207_L6.3mm_D2.5mm_P7.62mm_Horizontal, F.Cu at (211.0, 122.4)
- added R249: 100R, Resistor_THT:R_Axial_DIN0207_L6.3mm_D2.5mm_P7.62mm_Horizontal, F.Cu at (211.0, 130.7)
- added R250: 100R, Resistor_THT:R_Axial_DIN0207_L6.3mm_D2.5mm_P7.62mm_Horizontal, F.Cu at (211.0, 135.7)
- added U201: TL072, Package_DIP:DIP-8_W7.62mm_LongPads, F.Cu at (151.9, 90.0)
- added U202: TL072, Package_DIP:DIP-8_W7.62mm_LongPads, F.Cu at (151.9, 104.0)
- added U203: TL072, Package_DIP:DIP-8_W7.62mm_LongPads, F.Cu at (151.9, 117.3)
- added U204: TL072, Package_DIP:DIP-8_W7.62mm_LongPads, F.Cu at (151.9, 130.7)
- added U205: TL072, Package_DIP:DIP-8_W7.62mm_LongPads, F.Cu at (190.7, 90.6)
- added U206: TL072, Package_DIP:DIP-8_W7.62mm_LongPads, F.Cu at (190.7, 104.0)
- added U207: TL072, Package_DIP:DIP-8_W7.62mm_LongPads, F.Cu at (190.7, 117.3)
- added U208: TL072, Package_DIP:DIP-8_W7.62mm_LongPads, F.Cu at (190.7, 130.7)
Routing:
- net VEE: track 0.00 -> 271.6 mm
- net VCC: track 0.00 -> 233.2 mm
- net PU13: track 0.00 -> 94.3 mm
- net PU14: track 0.00 -> 91.9 mm
- net PU15: track 0.00 -> 85.6 mm
- net PU16: track 0.00 -> 81.7 mm
- net PU10: track 0.00 -> 76.4 mm, vias 0 -> 1
- net LINE08: track 0.00 -> 75.8 mm, vias 0 -> 1
- net PU09: track 0.00 -> 75.5 mm, vias 0 -> 1
- net PU11: track 0.00 -> 75.3 mm, vias 0 -> 1
- net LINE07: track 0.00 -> 73.7 mm, vias 0 -> 1
- net PU12: track 0.00 -> 73.1 mm, vias 0 -> 1
- net LINE06: track 0.00 -> 63.3 mm, vias 0 -> 1
- net PU07: track 0.00 -> 62.3 mm
- net LINE05: track 0.00 -> 62.1 mm, vias 0 -> 1
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- added copper zone on B.Cu, net GNDA
- added copper zone on F.Cu, net GNDA
Other:
- board outline added: 140 x 100 mm
- copper layers 0 -> 2
- board text added: "16 Channel CP70-pickup Amplifier Version 0.1 E.vd.Oetelaar May 30 2025"
- board text added: "Ch-01 Ch-02 Ch-03 Ch-04"
- board text added: "Ch-05 Ch-06 Ch-07 Ch-08"
- board text added: "Ch-09 Ch-10 Ch-11 Ch-12"
- board text added: "Ch-13 Ch-14 Ch-15 Ch-16"
- board text added: "GND"
- board text added: "GND GND"
- board text added: "V-MIN (VEE)"
- board text added: "VCC VCC"
- board text added: "VPLUS (VCC)"
