File: kicad_project/CP70_preamp/CP70_preamp.kicad_sch (KiCad schematic)
At the start: 0 parts

Commit message: design of 16 channel pre amp, including circuit board, ordered. Gerbers in repository.
Other:
- added sheet single_preamp_board (single_preamp.kicad_sch)
Changed lines of the file:
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@@
 		(company "POM (Eindhoven)")
+	)
+	(sheet
+		(at 143.51 27.94)
+		(size 71.12 52.07)
+		(exclude_from_sim no)
+		(in_bom yes)
+		(on_board yes)
+		(dnp no)
+		(fields_autoplaced yes)
+		(stroke
+			(width 0.1524)
+			(type solid)
+		)
+		(fill
+			(color 0 0 0 0.0000)
+		)
+		(property "Sheetname" "single_preamp_board"
+			(at 143.51 27.2284 0)
+			(effects
+				(font
+					(size 1.27 1.27)
+				)
+				(justify left bottom)
+			)
+		)
+		(property "Sheetfile" "single_preamp.kicad_sch"
+			(at 143.51 80.5946 0)
+			(effects
+				(font
+					(size 1.27 1.27)
+				)
+				(justify left top)
+			)
+		)
+		(instances
+			(project "CP70_preamp"
+				(path "/ea365a6d-81e4-484e-bf26-b7962246143f"
+					(page "2")
+				)
+			)
+		)
 	)
 	(sheet_instances
